File: Hardware/OpenMowerMainboard/OpenMowerMainboard.kicad_pcb (KiCad board)
At the start: 2 copper layers, 247.1 x 170 mm, 174 parts, among them IC1 74ALVC164245DGG,11, IC2 TSC101CILT, IC3 MAX20405AFOF_VY+T, J1 Conn_02x11_Top_Bottom, J10 Conn_01x05, J11 Conn_01x03_Male, J12 Conn_01x03_Male, J13 Conn_01x03_Male, J14 Conn_01x03_Male, J16 Conn_01x08, J17 Conn_01x02, J18 Conn_01x02, J19 Conn_01x04, J20 Conn_01x10_Female, J21 Raspberry_Pi_2_3, J22 Conn_02x04_Odd_Even, J23 Conn_01x08, J3 Conn_01x02, J4 Conn_01x05, J5 Conn_01x04, J51 Conn_01x04, J6 Conn_01x04, J7 Conn_01x04, J8 Conn_01x04, J9 Conn_01x04, M1 Fan, Q13 BSS138, Q14 BSS138, Q15 BSS138, Q16 BSS138, Q3 BSS138, Q5 BSS138, Q6 Q_PMOS_GDS, SW1 MK-11C04-G013, SW2 DA-01BP, U1 DNP, U10 74HC4051, U11 Pico, U2 MCP604, U3 SIP32509DT, U4 xESC2, U5 xESC2, U6 xESC2, U7 SN74LV1T34DBV, U9 74HC4051

Commit message: mainboard: turbocase compatibility
- Mounting holes for mounting PCB in case
- Raspberry Pi 4 footprint for turbocase connector cutouts
- Raspberry Pi 4 mounting hole footprint changed
Parts:
- added ?: , , F.Cu at (59.9, 132.3)
- added ?: , , F.Cu at (168.6, 146.8)
- added ?: , , F.Cu at (220.4, 113.2)
- added H1: MountingHole_Pad, MountingHole:MountingHole_2.5mm_Pad_Via, F.Cu at (301.8, 5.00)
- added H2: MountingHole_Pad, MountingHole:MountingHole_2.5mm_Pad_Via, F.Cu at (182.4, 62.6)
- added H3: MountingHole_Pad, MountingHole:MountingHole_2.5mm_Pad_Via, F.Cu at (58.8, 61.4)
- added H3: MountingHole_Pad, MountingHole:MountingHole_2.5mm_Pad_Via, F.Cu at (59.9, 132.3)
- added H3: MountingHole_Pad, MountingHole:MountingHole_2.5mm_Pad_Via, F.Cu at (168.6, 146.8)
- added H4: MountingHole_Pad, MountingHole:MountingHole_2.5mm_Pad_Via, F.Cu at (294.6, 162.6)
- added H4: MountingHole_Pad, MountingHole:MountingHole_2.5mm_Pad_Via, F.Cu at (221.7, 114.5)
- added RP?: Raspberry_Pi_2_3, rpi-footprints:raspberrypi_2_3, F.Cu at (245.7, 104.1)
- MH1, MH2, MH3, MH4, MH5, MH6, MH7, MH8: footprint MountingHole:MountingHole_2.7mm_M2.5 -> MountingHole:MountingHole_2.7mm_M2.5_Pad
Routing:
- net GND: vias 595 -> 597
Other:
- board size 247.1 x 170 mm -> 251.2 x 170 mm
